Commit message: rename custom bot to lw_mse6_bot

File: urdf/lw_mse6_bot.xacro (robot description, xacro)
@@ -65,5 +65,5 @@
             <origin xyz="0.0 0.0 0.0" rpy="0.0 0.0 0.0"/>
             <geometry>
-                <mesh filename="package://udacity_bot/meshes/new_mse6_tex.dae"/>
+                <mesh filename="package://udacity_bot/meshes/lw_mse6_chassis.dae"/>
             </geometry>
         </visual>
@@ -148,23 +148,4 @@
         </collision>
     </link>
-    <!-- <link name="body">
-        <inertial>
-            <origin xyz="0.0 0.0 0.0" rpy="0.0 0.0 0.0"/>
-            <mass value="0.1"/>
-            <inertia ixx="0.0000001" ixy="0.0" ixz="0.0" iyy="0.0000001" iyz="0.0" izz="0.0000001"/>
-        </inertial>
-        <visual name="">
-            <origin xyz="0.0 0.0 0.0" rpy="0.0 0.0 0.0"/>
-            <geometry>
-                <mesh filename="package://udacity_bot/meshes/new_mse6_tex.dae"/>
-            </geometry>
-        </visual>
-        <collision>
-            <origin xyz="0.0 0.0 0.0" rpy="0.0 0.0 0.0"/>
-            <geometry>
-                <box size="0.1 0.1 0.1"/>
-            </geometry>
-        </collision>
-    </link> -->
     <link name="camera">
         <inertial>

File: urdf/macros.xacro (robot description, xacro)
@@ -1,4 +1,4 @@
 <?xml version="1.0" encoding="UTF-8"?>
-<robot name="lw_udacity_bot_macros"
+<robot name="lw_mse6_bot_macros"
     xmlns:xacro="http://www.ros.org/wiki/xacro">
     <xacro:macro name="wheel" params="lr">

Commit message: fix(mse6_bot collision model): adjust collision model of mse6 bot using mesh; increase min range sen

File: urdf/lw_mse6_bot.xacro (robot description, xacro)
@@ -58,7 +58,7 @@
         <pose>0 0 ${wheelRadius} 0 0 0</pose>
         <inertial>
-            <origin xyz="0.0 0.0 0.0" rpy="0.0 0.0 0.0"/>
-            <mass value="0.1"/>
-            <inertia ixx="0.0000001" ixy="0.0" ixz="0.0" iyy="0.0000001" iyz="0.0" izz="0.0000001"/>
+            <mass value="18.0"/>
+            <origin xyz="0.0 0 0" rpy="0 0 0"/>
+            <inertia ixx="0.1" ixy="0" ixz="0" iyy="0.1" iyz="0" izz="0.1"/>
         </inertial>
         <visual name="">
@@ -68,8 +68,13 @@
             </geometry>
         </visual>
-        <collision>
+        <collision name='collision'>
+            <!--  dims x: [-0.3 ... 0.375] y: [-0.15 ... 0.15] z: [ -0.056 ... 0.18 ] -->
+            <!--<origin xyz="0.0375 0 0.062" rpy="0 0 0"/>
+            <geometry>
+                <box size="0.675 0.3 0.236"/>
+            </geometry>-->
             <origin xyz="0.0 0.0 0.0" rpy="0.0 0.0 0.0"/>
             <geometry>
-                <box size="0.1 0.1 0.1"/>
+                <mesh filename="package://udacity_bot/meshes/lw_mse6_chassis.dae"/>
             </geometry>
         </collision>
